Commit message: added imu link, minor bug fixes related to paths and gazebo plugins

File: tortoisebot_description/models/urdf/tortoisebot_simple.xacro (robot description, xacro)
@@ -4,5 +4,4 @@
 <xacro:include filename="$(find tortoisebot_gazebo)/gazebo/tortoisebot_physics.gazebo" />
 <xacro:include filename="$(find tortoisebot_gazebo)/gazebo/tortoisebot_plugins.gazebo" />
-<xacro:include filename="$(find ttb_description)/models/urdf/tortoisebot_simple.gazebo" />
 <link name="base_link">
   <inertial>
@@ -138,4 +137,5 @@
   </collision>
 </link>
+<link name="imu_link"/>
 <joint name="wheel_left_joint" type="continuous">
   <origin xyz="-0.000197 0.0778 0.032453" rpy="0 0 0"/>
@@ -170,3 +170,8 @@
   <child link="castor_wheel"/>
 </joint>
+<joint name="imu_joint" type="fixed">
+  <origin xyz="0.0 0.0 0.11" rpy="0 0 0"/>
+  <parent link="base_link"/>
+  <child link="imu_link"/>
+</joint>
 </robot>
